File: spark-console-pcb.kicad_sch (KiCad schematic)
At the start: 0 parts

Commit message: Finished first version of schematics
Parts:
- added BZ1: Buzzer, symbol Device:Buzzer
- added C1: 100n, symbol Device:C
- added C2, C3: 22pF, symbol Device:C
- added C4: 100uF, symbol Device:C_Polarized
- added D1: POWER LED, symbol Device:LED
- added D2, D3, D4, D5: USER LED, symbol Device:LED
- added J1: USB_B, symbol Connector:USB_B
- added J2: PROGRAM, symbol Connector:Conn_01x05_Male
- added R1: 10k, symbol Device:R
- added R2, R3, R4, R5, R6, R7: 470, symbol Device:R
- added R8, R9: R, symbol Device:R
- added SW1, SW2, SW3, SW4, SW5, SW6, SW7: SW_Push, symbol Switch:SW_Push
- added U1: ATmega328P-P, Package_DIP:DIP-28_W7.62mm, symbol MCU_Microchip_ATmega:ATmega328P-P
- added U2, U3: MAX7221xWG, Package_SO:SOIC-24W_7.5x15.4mm_P1.27mm, symbol Driver_LED:MAX7221xWG
- added U4: HL-M1388BRPG, symbol spark-console:HL-M1388BRPG
- added Y1: Crystal, symbol Device:Crystal
Connections:
- new net: D4.2 (A), R6.1
- new net: D3.2 (A), R5.1
- new net: U2.3 (DIG_4), U4.1
- new net: U2.8 (DIG_7), U4.10
- new net: U3.8 (DIG_7), U4.11
- new net: U2.14 (SEG_A), U3.14 (SEG_A), U4.12
- new net: U2.21 (SEG_E), U3.21 (SEG_E), U4.13
- new net: U3.7 (DIG_3), U4.14
- new net: U2.7 (DIG_3), U4.15
- new net: U2.15 (SEG_F), U3.15 (SEG_F), U4.16
- new net: U3.6 (DIG_2), U4.17
- new net: U2.6 (DIG_2), U4.18
- new net: U2.17 (SEG_G), U3.17 (SEG_G), U4.19
- new net: U3.3 (DIG_4), U4.2
- new net: U3.11 (DIG_1), U4.20
- new net: U2.11 (DIG_1), U4.21
- new net: U2.22 (SEG_DP), U3.22 (SEG_DP), U4.22
- new net: U3.2 (DIG_0), U4.23
- new net: U2.2 (DIG_0), U4.24
- new net: U2.23 (SEG_D), U3.23 (SEG_D), U4.3
- new net: U2.10 (DIG_5), U4.4
- new net: U3.10 (DIG_5), U4.5
- new net: U2.20 (SEG_C), U3.20 (SEG_C), U4.6
- new net: U2.5 (DIG_6), U4.7
- new net: U3.5 (DIG_6), U4.8
- new net: U2.16 (SEG_B), U3.16 (SEG_B), U4.9
- new net: D2.2 (A), R4.1
- new net: R4.2, U1.13 (PD7)
- new net: J2.3 (Pin_3), U1.3 (PD1)
- new net: J2.4 (Pin_4), U1.2 (PD0)
- new net: D5.2 (A), R7.1
- new net: R7.2, U1.6 (PD4)
- new net: U2.24 (DOUT), U3.1 (DIN)
- new net: R9.2, U3.18 (ISET)
- new net: C2.1, U1.9 (XTAL1/PB6), Y1.2
- new net: C3.1, U1.10 (XTAL2/PB7), Y1.1
- new net: R6.2, U1.11 (PD5)
- new net: R5.2, U1.12 (PD6)
- new net: D1.2 (A), R2.1
- new net: BZ1.1 (-), R3.1
- new net: R8.2, U2.18 (ISET)
- new net BTN_A: SW6.2, U1.24 (PC1)
- new net BTN_B: SW7.2, U1.23 (PC0)
- new net BTN_DOWN: SW5.2, U1.25 (PC2)
- new net BTN_LEFT: SW1.2, U1.28 (PC5)
- new net BTN_RIGHT: SW2.2, U1.27 (PC4)
- new net BTN_UP: SW4.2, U1.26 (PC3)
- new net BUZZER: R3.2, U1.5 (PD3)
- new net CLK: U1.19 (PB5), U2.13 (CLK), U3.13 (CLK)
- new net CS: U1.16 (PB2), U2.12 (~CS), U3.12 (~CS)
- new net GND: BZ1.2 (+), C1.2, C2.2, C3.2, C4.2, D1.1 (K), D2.1 (K), D3.1 (K), D4.1 (K), D5.1 (K), J1.4 (GND), J1.5 (Shield), J2.1 (Pin_1), SW1.1, SW2.1, SW3.1, SW4.1, SW5.1, SW6.1, SW7.1, U1.22 (GND), U1.8 (GND), U2.4 (GND), U2.9 (GND), U3.4 (GND), U3.9 (GND)
- new net MOSI: U1.17 (PB3), U2.1 (DIN)
- new net RESET: J2.2 (Pin_2), R1.1, SW3.2, U1.1 (~RESET~/PC6)
- new net VCC: C1.1, C4.1, J1.1 (VBUS), J2.5 (Pin_5), R1.2, R2.2, R8.1, R9.1, U1.20 (AVCC), U1.7 (VCC), U2.19 (V+), U3.19 (V+)
- no-connect marks 0 -> 8
