File: spark-console-pcb.kicad_sch (KiCad schematic)
At the start: 33 parts, among them J1 USB_B, J2 PROGRAM, SW1 SW_Push, SW2 SW_Push, SW3 SW_Push, SW4 SW_Push, SW5 SW_Push, SW6 SW_Push, SW7 SW_Push, U1 ATmega328P-P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

Commit message: Associated symbols and footprints
Parts:
- BZ1: footprint (none) -> Buzzer_Beeper:Buzzer_15x7.5RM7.6
- C1, C2, C3: footprint (none) -> Capacitor_THT:C_Disc_D4.7mm_W2.5mm_P5.00mm
- C4: footprint (none) -> Capacitor_THT:CP_Radial_D6.3mm_P2.50mm
- D1, D2, D3, D4, D5: footprint (none) -> LED_THT:LED_D3.0mm
- J1: footprint (none) -> Connector_USB:USB_B_OST_USB-B1HSxx_Horizontal
- J2: footprint (none) -> Connector_PinHeader_2.54mm:PinHeader_1x05_P2.54mm_Horizontal
- R1, R2, R3, R4, R5, R6, R7, R8, R9: footprint (none) -> Resistor_THT:R_Axial_DIN0204_L3.6mm_D1.6mm_P7.62mm_Horizontal
- SW1, SW2, SW3, SW4, SW5, SW6, SW7: footprint (none) -> Button_Switch_THT:SW_PUSH_6mm_H5mm
- U4: footprint (none) -> spark-console:HL-M1388BRPG
- Y1: footprint (none) -> Crystal:Crystal_HC49-4H_Vertical

Commit message: Fix MAX7221 footprint
Parts:
- removed U2, U3: MAX7221xWG, Package_SO:SOIC-24W_7.5x15.4mm_P1.27mm, symbol Driver_LED:MAX7221xWG
- added U2, U3: MAX7221xNG, Package_DIP:DIP-24_W7.62mm, symbol Driver_LED:MAX7221xNG
Connections:
- net CLK: now also U2.13 (CLK), U3.13 (CLK)
- net CS: now also U2.12 (~CS), U3.12 (~CS)
- net GND: now also U2.4 (GND), U2.9 (GND), U3.4 (GND), U3.9 (GND)
- net MOSI: now also U2.1 (DIN)
- net VCC: now also U2.19 (V+), U3.19 (V+)
- net at U4.1: now also U2.3 (DIG_4)
- net at U4.10: now also U2.8 (DIG_7)
- net at U4.11: now also U3.8 (DIG_7)
- net at U4.12: now also U2.14 (SEG_A), U3.14 (SEG_A)
- net at U4.13: now also U2.21 (SEG_E), U3.21 (SEG_E)
- net at U4.14: now also U3.7 (DIG_3)
- net at U4.15: now also U2.7 (DIG_3)
- net at U4.16: now also U2.15 (SEG_F), U3.15 (SEG_F)
- net at U4.17: now also U3.6 (DIG_2)
- net at U4.18: now also U2.6 (DIG_2)
- net at U4.19: now also U2.17 (SEG_G), U3.17 (SEG_G)
- net at U4.2: now also U3.3 (DIG_4)
- net at U4.20: now also U3.11 (DIG_1)
- net at U4.21: now also U2.11 (DIG_1)
- net at U4.22: now also U2.22 (SEG_DP), U3.22 (SEG_DP)
- net at U4.23: now also U3.2 (DIG_0)
- net at U4.24: now also U2.2 (DIG_0)
- net at U4.3: now also U2.23 (SEG_D), U3.23 (SEG_D)
- net at U4.4: now also U2.10 (DIG_5)
- net at U4.5: now also U3.10 (DIG_5)
- net at U4.6: now also U2.20 (SEG_C), U3.20 (SEG_C)
- net at U4.7: now also U2.5 (DIG_6)
- net at U4.8: now also U3.5 (DIG_6)
- net at U4.9: now also U2.16 (SEG_B), U3.16 (SEG_B)
- net at R9.2: now also U3.18 (ISET)
- net at R8.2: now also U2.18 (ISET)
- new net: U2.24 (DOUT), U3.1 (DIN)
Changed lines of the file:
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@@
     (pin "5")
   )
-  (symbol (lib_id "Driver_LED:MAX7221xWG") (at 173.99 50.165 0) (unit 1)
+  (symbol (lib_id "Driver_LED:MAX7221xNG") (at 173.99 50.165 0) (unit 1)
     (in_bom yes) (on_board yes)
-    (property "Reference" "U2" (id 0) (at 182.245 22.9828 0))
-    (property "Value" "MAX7221xWG" (id 1) (at 181.61 25.2815 0))
-    (property "Footprint" "Package_SO:SOIC-24W_7.5x15.4mm_P1.27mm" (id 2) (at 172.72 48.895 0)
+    (property "Reference" "U2" (id 0) (at 182.245 22.3478 0))
+    (property "Value" "MAX7221xNG" (id 1) (at 183.515 24.6465 0))
+    (property "Footprint" "Package_DIP:DIP-24_W7.62mm" (id 2) (at 172.72 48.895 0)
       (effects (font (size 1.27 1.27)) hide)
     )
@@
     (pin "9")
   )
-  (symbol (lib_id "Driver_LED:MAX7221xWG") (at 173.99 109.22 0) (unit 1)
+  (symbol (lib_id "Driver_LED:MAX7221xNG") (at 173.99 109.22 0) (unit 1)
     (in_bom yes) (on_board yes)
-    (property "Reference" "U3" (id 0) (at 180.975 134.1078 0))
-    (property "Value" "MAX7221xWG" (id 1) (at 180.975 136.4065 0))
-    (property "Footprint" "Package_SO:SOIC-24W_7.5x15.4mm_P1.27mm" (id 2) (at 172.72 107.95 0)
+    (property "Reference" "U3" (id 0) (at 182.245 81.4028 0))
+    (property "Value" "MAX7221xNG" (id 1) (at 183.515 83.7015 0))
+    (property "Footprint" "Package_DIP:DIP-24_W7.62mm" (id 2) (at 172.72 107.95 0)
       (effects (font (size 1.27 1.27)) hide)
     )
@@
       (reference "U1") (unit 1) (value "ATmega328P-P") (footprint "Package_DIP:DIP-28_W7.62mm")
     )
-    (path "/ea4171ed-fb2e-4efe-8081-6064f6577fea"
-      (reference "U2") (unit 1) (value "MAX7221xWG") (footprint "Package_SO:SOIC-24W_7.5x15.4mm_P1.27mm")
-    )
-    (path "/52c60fb2-cd82-4d0e-ad0e-a21304f344a9"
-      (reference "U3") (unit 1) (value "MAX7221xWG") (footprint "Package_SO:SOIC-24W_7.5x15.4mm_P1.27mm")
+    (path "/5b91a266-99ea-47eb-bd01-5f2f3a6703d6"
+      (reference "U2") (unit 1) (value "MAX7221xNG") (footprint "Package_DIP:DIP-24_W7.62mm")
+    )
+    (path "/f21041ad-7445-434f-acab-b2b55712c350"
+      (reference "U3") (unit 1) (value "MAX7221xNG") (footprint "Package_DIP:DIP-24_W7.62mm")
     )
     (path "/1d8a8d3c-8584-4e83-ae2b-bf0ac23efe2a"

Commit message: Added first version of PCB
Changed lines of the file:
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@@
   (symbol (lib_id "spark-console:HL-M1388BRPG") (at 224.79 36.195 0) (mirror x) (unit 1)
     (in_bom yes) (on_board yes) (fields_autoplaced)
-    (property "Reference" "U4" (id 0) (at 241.1476 15.0326 0))
-    (property "Value" "HL-M1388BRPG" (id 1) (at 241.1476 17.3313 0))
-    (property "Footprint" "spark-console:HL-M1388BRPG" (id 2) (at 265.43 15.875 0)
+    (property "Reference" "U4" (id 0) (at 241.1476 57.3574 0))
+    (property "Value" "HL-M1388BRPG" (id 1) (at 241.1476 55.0587 0))
+    (property "Footprint" "spark-console:HL-M1388BRPG" (id 2) (at 265.43 56.515 0)
       (effects (font (size 1.27 1.27)) hide)
     )
-    (property "Datasheet" "" (id 3) (at 265.43 15.875 0)
+    (property "Datasheet" "" (id 3) (at 265.43 56.515 0)
       (effects (font (size 1.27 1.27)) hide)
     )

Commit message: Changes from lazerninja
Parts:
- J1: footprint Connector_USB:USB_B_OST_USB-B1HSxx_Horizontal -> Connector_USB:USB_Micro-B_Wuerth_614105150721_Vertical
- SW1, SW2, SW4, SW5, SW6, SW7: footprint Button_Switch_THT:SW_PUSH_6mm_H5mm -> Button_Switch_THT:SW_PUSH-12mm
- SW3: footprint Button_Switch_THT:SW_PUSH_6mm_H5mm -> Button_Switch_THT:SW_PUSH_6mm
Changed lines of the file:
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@@
       (effects (font (size 1.27 1.27)) (justify right))
     )
-    (property "Footprint" "Button_Switch_THT:SW_PUSH_6mm_H5mm" (id 2) (at 17.78 33.655 0)
+    (property "Footprint" "Button_Switch_THT:SW_PUSH-12mm" (id 2) (at 17.78 33.655 0)
       (effects (font (size 1.27 1.27)) hide)
     )
@@
       (effects (font (size 1.27 1.27)) (justify right))
     )
-    (property "Footprint" "Button_Switch_THT:SW_PUSH_6mm_H5mm" (id 2) (at 26.035 33.655 0)
+    (property "Footprint" "Button_Switch_THT:SW_PUSH-12mm" (id 2) (at 26.035 33.655 0)
       (effects (font (size 1.27 1.27)) hide)
     )
@@
       (effects (font (size 1.27 1.27)) (justify right))
     )
-    (property "Footprint" "Button_Switch_THT:SW_PUSH_6mm_H5mm" (id 2) (at 27.305 66.675 0)
+    (property "Footprint" "Button_Switch_THT:SW_PUSH_6mm" (id 2) (at 27.305 66.675 0)
       (effects (font (size 1.27 1.27)) hide)
     )
@@
       (effects (font (size 1.27 1.27)) (justify right))
     )
-    (property "Footprint" "Button_Switch_THT:SW_PUSH_6mm_H5mm" (id 2) (at 34.29 33.655 0)
+    (property "Footprint" "Button_Switch_THT:SW_PUSH-12mm" (id 2) (at 34.29 33.655 0)
       (effects (font (size 1.27 1.27)) hide)
     )
@@
       (effects (font (size 1.27 1.27)) (justify right))
     )
-    (property "Footprint" "Button_Switch_THT:SW_PUSH_6mm_H5mm" (id 2) (at 42.545 33.655 0)
+    (property "Footprint" "Button_Switch_THT:SW_PUSH-12mm" (id 2) (at 42.545 33.655 0)
       (effects (font (size 1.27 1.27)) hide)
     )
@@
       (effects (font (size 1.27 1.27)) (justify right))
     )
-    (property "Footprint" "Button_Switch_THT:SW_PUSH_6mm_H5mm" (id 2) (at 50.8 33.02 0)
+    (property "Footprint" "Button_Switch_THT:SW_PUSH-12mm" (id 2) (at 50.8 33.02 0)
       (effects (font (size 1.27 1.27)) hide)
     )
@@
       (effects (font (size 1.27 1.27)) (justify right))
     )
-    (property "Footprint" "Button_Switch_THT:SW_PUSH_6mm_H5mm" (id 2) (at 58.42 33.02 0)
+    (property "Footprint" "Button_Switch_THT:SW_PUSH-12mm" (id 2) (at 58.42 33.02 0)
       (effects (font (size 1.27 1.27)) hide)
     )
@@
     (property "Reference" "J1" (id 0) (at 31.877 162.3018 0))
     (property "Value" "USB_B" (id 1) (at 31.877 164.6005 0))
-    (property "Footprint" "Connector_USB:USB_B_OST_USB-B1HSxx_Horizontal" (id 2) (at 34.29 174.625 0)
+    (property "Footprint" "Connector_USB:USB_Micro-B_Wuerth_614105150721_Vertical" (id 2) (at 34.29 174.625 0)
       (effects (font (size 1.27 1.27)) hide)
     )
@@
     )
     (path "/398b1e3b-1edb-486f-9f4d-113a8bb0afce"
-      (reference "J1") (unit 1) (value "USB_B") (footprint "Connector_USB:USB_B_OST_USB-B1HSxx_Horizontal")
+      (reference "J1") (unit 1) (value "USB_B") (footprint "Connector_USB:USB_Micro-B_Wuerth_614105150721_Vertical")
     )
     (path "/42139282-2749-45fb-9938-ce26eb944796"
@@
     )
     (path "/f6c33365-898a-40c6-b607-76da91f90276"
-      (reference "SW1") (unit 1) (value "SW_Push") (footprint "Button_Switch_THT:SW_PUSH_6mm_H5mm")
+      (reference "SW1") (unit 1) (value "SW_Push") (footprint "Button_Switch_THT:SW_PUSH-12mm")
     )
     (path "/0178c8eb-9d23-497d-8277-13ba6952c3b1"
-      (reference "SW2") (unit 1) (value "SW_Push") (footprint "Button_Switch_THT:SW_PUSH_6mm_H5mm")
+      (reference "SW2") (unit 1) (value "SW_Push") (footprint "Button_Switch_THT:SW_PUSH-12mm")
     )
     (path "/4f447cf9-9f61-4908-962a-0d5665e9e470"
-      (reference "SW3") (unit 1) (value "SW_Push") (footprint "Button_Switch_THT:SW_PUSH_6mm_H5mm")
+      (reference "SW3") (unit 1) (value "SW_Push") (footprint "Button_Switch_THT:SW_PUSH_6mm")
     )
     (path "/064570d0-6f75-4f08-97db-1bee6579bdbd"
-      (reference "SW4") (unit 1) (value "SW_Push") (footprint "Button_Switch_THT:SW_PUSH_6mm_H5mm")
+      (reference "SW4") (unit 1) (value "SW_Push") (footprint "Button_Switch_THT:SW_PUSH-12mm")
     )
     (path "/e5b647e2-cde7-4b1f-ba9e-5196d43328a8"
-      (reference "SW5") (unit 1) (value "SW_Push") (footprint "Button_Switch_THT:SW_PUSH_6mm_H5mm")
+      (reference "SW5") (unit 1) (value "SW_Push") (footprint "Button_Switch_THT:SW_PUSH-12mm")
     )
     (path "/29d03701-0878-41ce-84c7-134df427a4ca"
-      (reference "SW6") (unit 1) (value "SW_Push") (footprint "Button_Switch_THT:SW_PUSH_6mm_H5mm")
+      (reference "SW6") (unit 1) (value "SW_Push") (footprint "Button_Switch_THT:SW_PUSH-12mm")
     )
     (path "/4754d30a-0680-47cd-a68d-86f542bd01eb"
-      (reference "SW7") (unit 1) (value "SW_Push") (footprint "Button_Switch_THT:SW_PUSH_6mm_H5mm")
+      (reference "SW7") (unit 1) (value "SW_Push") (footprint "Button_Switch_THT:SW_PUSH-12mm")
     )
     (path "/686dcfb3-3ea5-4639-8df1-cda088d2b2e2"
