File: spark-console-pcb.kicad_pcb (KiCad board)
At the start: 0 parts

Commit message: Added first version of PCB
Parts:
- added BZ1: Buzzer, Buzzer_Beeper:Buzzer_15x7.5RM7.6, B.Cu at (125.2, 77.8)
- added C1: 100n, Capacitor_THT:C_Disc_D4.7mm_W2.5mm_P5.00mm, F.Cu at (179.2, 92.5)
- added C2: 22pF, Capacitor_THT:C_Disc_D4.7mm_W2.5mm_P5.00mm, F.Cu at (156.8, 118.1)
- added C3: 22pF, Capacitor_THT:C_Disc_D4.7mm_W2.5mm_P5.00mm, F.Cu at (141.8, 118.1)
- added C4: 100uF, Capacitor_THT:CP_Radial_D6.3mm_P2.50mm, F.Cu at (190.0, 105.0)
- added D1: POWER LED, LED_THT:LED_D3.0mm, F.Cu at (182.5, 72.5)
- added D2: USER LED, LED_THT:LED_D3.0mm, F.Cu at (146.3, 64.4)
- added D3: USER LED, LED_THT:LED_D3.0mm, F.Cu at (141.3, 64.4)
- added D4: USER LED, LED_THT:LED_D3.0mm, F.Cu at (151.3, 64.4)
- added D5: USER LED, LED_THT:LED_D3.0mm, F.Cu at (156.3, 64.4)
- added J1: USB_B, Connector_USB:USB_B_OST_USB-B1HSxx_Horizontal, F.Cu at (190.2, 91.2)
- added J2: PROGRAM, Connector_PinHeader_2.54mm:PinHeader_1x05_P2.54mm_Horizontal, F.Cu at (100.0, 97.6)
- added R1: 10k, Resistor_THT:R_Axial_DIN0204_L3.6mm_D1.6mm_P7.62mm_Horizontal, F.Cu at (128.8, 112.5)
- added R2: 470, Resistor_THT:R_Axial_DIN0204_L3.6mm_D1.6mm_P7.62mm_Horizontal, F.Cu at (190.0, 73.7)
- added R3: 470, Resistor_THT:R_Axial_DIN0204_L3.6mm_D1.6mm_P7.62mm_Horizontal, F.Cu at (119.1, 73.6)
- added R4: 470, Resistor_THT:R_Axial_DIN0204_L3.6mm_D1.6mm_P7.62mm_Horizontal, F.Cu at (132.5, 66.2)
- added R5: 470, Resistor_THT:R_Axial_DIN0204_L3.6mm_D1.6mm_P7.62mm_Horizontal, F.Cu at (130.0, 66.2)
- added R6: 470, Resistor_THT:R_Axial_DIN0204_L3.6mm_D1.6mm_P7.62mm_Horizontal, F.Cu at (172.5, 71.2)
- added R7: 470, Resistor_THT:R_Axial_DIN0204_L3.6mm_D1.6mm_P7.62mm_Horizontal, F.Cu at (175.0, 71.2)
- added R8: R, Resistor_THT:R_Axial_DIN0204_L3.6mm_D1.6mm_P7.62mm_Horizontal, F.Cu at (146.8, 87.6)
- added R9: R, Resistor_THT:R_Axial_DIN0204_L3.6mm_D1.6mm_P7.62mm_Horizontal, F.Cu at (145.4, 71.6)
- added SW1: SW_Push, Button_Switch_THT:SW_PUSH_6mm_H5mm, F.Cu at (178.5, 100.8)
- added SW2: SW_Push, Button_Switch_THT:SW_PUSH_6mm_H5mm, F.Cu at (114.2, 100.8)
- added SW3: SW_Push, Button_Switch_THT:SW_PUSH_6mm_H5mm, F.Cu at (178.5, 110.2)
- added SW4: SW_Push, Button_Switch_THT:SW_PUSH_6mm_H5mm, F.Cu at (179.2, 80.8)
- added SW5: SW_Push, Button_Switch_THT:SW_PUSH_6mm_H5mm, F.Cu at (113.5, 80.8)
- added SW6: SW_Push, Button_Switch_THT:SW_PUSH_6mm_H5mm, F.Cu at (103.5, 90.8)
- added SW7: SW_Push, Button_Switch_THT:SW_PUSH_6mm_H5mm, F.Cu at (123.5, 90.8)
- added U1: ATmega328P-P, Package_DIP:DIP-28_W7.62mm, B.Cu at (168.2, 114.4)
- added U2: MAX7221xNG, Package_DIP:DIP-24_W7.62mm, F.Cu at (136.3, 97.4)
- added U3: MAX7221xNG, Package_DIP:DIP-24_W7.62mm, F.Cu at (136.3, 85.4)
- added U4: HL-M1388BRPG, spark-console:HL-M1388BRPG, F.Cu at (149.4, 86.6)
- added Y1: Crystal, Crystal:Crystal_HC49-4H_Vertical, B.Cu at (146.8, 118.1)
Routing:
- net GND: track 0.00 -> 328.7 mm
- net VCC: track 0.00 -> 209.9 mm
- net /RESET: track 0.00 -> 94.0 mm
- net Net-(J2-Pad4): track 0.00 -> 85.6 mm
- net /CLK: track 0.00 -> 84.5 mm
- net /BUZZER: track 0.00 -> 79.5 mm
- net Net-(J2-Pad3): track 0.00 -> 77.3 mm
- net /BTN_A: track 0.00 -> 61.5 mm
- net Net-(R6-Pad2): track 0.00 -> 57.7 mm
- net /BTN_DOWN: track 0.00 -> 57.0 mm
- net /BTN_RIGHT: track 0.00 -> 54.3 mm
- net Net-(R5-Pad2): track 0.00 -> 48.3 mm
- net Net-(U2-Pad8): track 0.00 -> 47.6 mm
- net /CS: track 0.00 -> 46.5 mm, vias 0 -> 1
- net Net-(R7-Pad2): track 0.00 -> 43.9 mm
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Other:
- board outline added: 105 x 57.5 mm
- copper layers 0 -> 2
